File: hardware/top-board/TubeDrivers.kicad_sch (KiCad schematic)
At the start: 17 parts, among them U5 TPIC6B595DWR, U6 TPIC6B595DWR, U7 TPIC6B595DWR, U8 TPIC6B595DWR

Commit message: Add provisional GZC9-A footprint and unblock top-board placement
Parts:
- V1, V2, V3, V4: footprint (none) -> Numitron:GZC9-A_B9A_Provisional; FootprintStatus HOLD: socket-tail measurements -> PROVISIONAL: 18 mm PCD, 0.5 mm terminal thickness, 2.5 mm h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
