File: hardware/top-board/ControlAndSensor.kicad_sch (KiCad schematic)
At the start: 27 parts, among them Q1 MMBT3904-7-F, U2 SN74AHCT125DR, U3 BH1750FVI-TR, U4 TLV809EA29DBZR

Commit message: Complete routed top-board prototype layout
Parts:
- U3: footprint (none) -> Numitron:ROHM_WSOF6I_BH1750_NoCenterPad; FootprintStatus HOLD: verify WSOF6I land pattern; no center-pad solder -> ROHM 0.25 x 0.55 mm six-land pattern; no center pad; top co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
Changed lines of the file:
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@@
           (instances (project "NumitronTop" (path "/89c4ac53-0d74-5f5d-9ed8-8226c02dc936/80c1f917-a0fd-5c73-9f82-08b8ac7ddbdb" (reference "R14") (unit 1)))))(wire (pts (xy 162.56 189.23) (xy 162.56 186.69)) (stroke (width 0.1524) (type default)))(global_label "+3V3" (shape input) (at 162.56 186.69 0) (effects (font (size 1.016 1.016)) (justify left) ))(wire (pts (xy 162.56 199.39) (xy 162.56 201.93)) (stroke (width 0.1524) (type default)))(global_label "BLANK_3V3" (shape input) (at 162.56 201.93 0) (effects (font (size 1.016 1.016)) (justify left) ))(text "STARTUP CONTRACT" (at 17.78 224.79 0) (effects (font (size 1.524 1.524)) (justify left top) ))(text "1. ARM low; configure SER/SRCK/RCK low and BLANK high.\n2. ARM high; clock 32 zero bits, pulse RCK with SRCK low.\n3. Load the desired frame; only then enable BLANK PWM.\n4. BLANK low = lit. A logic one in a drain bit lights a filament.\nStart with 100 kHz SPI mode 0; verify signals before raising speed." (at 17.78 232.41 0) (effects (font (size 1.27 1.27)) (justify left top) ))(text "AMBIENT LIGHT / 3.3 V I2C" (at 228.6 135.89 0) (effects (font (size 1.524 1.524)) (justify left top) ))(symbol (lib_id "Numitron:BH1750FVI") (at 350.52 177.8 0) (unit 1)
           (in_bom yes) (on_board yes) (dnp no)
- (property "Reference" "U3" (at 354.33 162.56 0) (effects (font (size 1.27 1.27)) (justify left) ))(property "Value" "BH1750FVI-TR" (at 354.33 165.1 0) (effects (font (size 1.27 1.27)) (justify left) ))(property "Footprint" "" (at 0 0 0) (effects (font (size 1.27 1.27))  hide))(property "Datasheet" "${KIPRJMOD}/../../datasheets/bh1750fvi.pdf" (at 0 0 0) (effects (font (size 1.27 1.27))  hide))(property "Description" "Ambient light sensor; 0x23 with ADDR low; WSOF6I exposed center must NOT be soldered" (at 0 0 0) (effects (font (size 1.27 1.27))  hide))(property "MPN" "BH1750FVI-TR" (at 0 0 0) (effects (font (size 1.27 1.27))  hide))(property "Manufacturer" "ROHM" (at 0 0 0) (effects (font (size 1.27 1.27))  hide))(property "FootprintStatus" "HOLD: verify WSOF6I land pattern; no center-pad solder" (at 0 0 0) (effects (font (size 1.27 1.27))  hide)) (pin "1") (pin "3") (pin "2") (pin "5") (pin "6") (pin "4")
+ (property "Reference" "U3" (at 354.33 162.56 0) (effects (font (size 1.27 1.27)) (justify left) ))(property "Value" "BH1750FVI-TR" (at 354.33 165.1 0) (effects (font (size 1.27 1.27)) (justify left) ))(property "Footprint" "Numitron:ROHM_WSOF6I_BH1750_NoCenterPad" (at 0 0 0) (effects (font (size 1.27 1.27))  hide))(property "Datasheet" "${KIPRJMOD}/../../datasheets/bh1750fvi.pdf" (at 0 0 0) (effects (font (size 1.27 1.27))  hide))(property "Description" "Ambient light sensor; 0x23 with ADDR low; WSOF6I exposed center must NOT be soldered" (at 0 0 0) (effects (font (size 1.27 1.27))  hide))(property "MPN" "BH1750FVI-TR" (at 0 0 0) (effects (font (size 1.27 1.27))  hide))(property "Manufacturer" "ROHM" (at 0 0 0) (effects (font (size 1.27 1.27))  hide))(property "FootprintStatus" "ROHM 0.25 x 0.55 mm six-land pattern; no center pad; top copper keepout" (at 0 0 0) (effects (font (size 1.27 1.27))  hide)) (pin "1") (pin "3") (pin "2") (pin "5") (pin "6") (pin "4")
           (instances (project "NumitronTop" (path "/89c4ac53-0d74-5f5d-9ed8-8226c02dc936/80c1f917-a0fd-5c73-9f82-08b8ac7ddbdb" (reference "U3") (unit 1)))))(wire (pts (xy 350.52 165.1) (xy 350.52 160.02)) (stroke (width 0.1524) (type default)))(global_label "+3V3" (shape input) (at 350.52 160.02 0) (effects (font (size 1.016 1.016)) (justify left) ))(wire (pts (xy 350.52 190.5) (xy 350.52 195.58)) (stroke (width 0.1524) (type default)))(global_label "GND" (shape input) (at 350.52 195.58 0) (effects (font (size 1.016 1.016)) (justify left) ))(wire (pts (xy 363.22 172.72) (xy 370.84 172.72)) (stroke (width 0.1524) (type default)))(global_label "SCL" (shape input) (at 370.84 172.72 0) (effects (font (size 1.016 1.016)) (justify left) ))(wire (pts (xy 363.22 177.8) (xy 370.84 177.8)) (stroke (width 0.1524) (type default)))(global_label "SDA" (shape input) (at 370.84 177.8 0) (effects (font (size 1.016 1.016)) (justify left) ))(symbol (lib_id "Numitron:TLV809EA29DBZ") (at 261.62 172.72 0) (unit 1)
           (in_bom yes) (on_board yes) (dnp no)
